Commit message: Update rover URDF with IMU, Camera, and Lidar positions and rotations

File: src/rover_description/urdf/rover.urdf.xacro (robot description, xacro)
@@ -56,18 +56,20 @@
     <parent link="base_link"/>
     <child link="bno055"/>
-    <origin xyz="0.05 0.0 0.05" rpy="0 0 0"/>
+    <!-- This configuration is based on my estimate for where the center of the chip is
+    the IMU is mounted in a right-handed X right Y forward configuration. -->
+    <origin xyz="-0.03928461 -0.050864 0.14345" rpy="0 0 ${pi/2}"/>
   </joint>
-  <link name="laser_frame">
+  <link name="lidar_frame">
     <visual>
       <geometry>
-        <cylinder radius="0.05" length="0.04"/>
+        <cylinder radius="0.061331" length="0.038040"/>
       </geometry>
-      <material name="black"/>
+      <material name="blue"/>
     </visual>
   </link>
-  <joint name="laser_joint" type="fixed">
+  <joint name="lidar_joint" type="fixed">
     <parent link="base_link"/>
     <child link="laser_frame"/>
-    <origin xyz="0.0 0.0 ${chassis_height/2 + 0.02}" rpy="0 0 0"/>
+    <origin xyz="0.0 0.043684 .19576183" rpy="0 ${22 * pi / 180} 0"/>
   </joint>
   <link name="camera_link">
@@ -76,5 +78,5 @@
         <box size="0.02 0.06 0.02"/>
       </geometry>
-      <material name="red"/>
+      <material name="blue"/>
     </visual>
   </link>
@@ -82,5 +84,5 @@
     <parent link="base_link"/>
     <child link="camera_link"/>
-    <origin xyz="${chassis_length/2 + 0.01} 0.0 0.08" rpy="0 0 0"/>
+    <origin xyz=".196296 .060 .135925" rpy="0 0 0"/>
   </joint>
   <link name="camera_link_optical"/>

Commit message: Configure synchronous lidar and camera launch, update accessories config layout, and fix URDF frame matching

File: src/rover_description/urdf/rover.urdf.xacro (robot description, xacro)
@@ -60,5 +60,5 @@
     <origin xyz="-0.03928461 -0.050864 0.14345" rpy="0 0 ${pi/2}"/>
   </joint>
-  <link name="lidar_frame">
+  <link name="rslidar">
     <visual>
       <geometry>
@@ -70,5 +70,5 @@
   <joint name="lidar_joint" type="fixed">
     <parent link="base_link"/>
-    <child link="laser_frame"/>
+    <child link="rslidar"/>
     <origin xyz="0.0 0.043684 .19576183" rpy="0 ${22 * pi / 180} 0"/>
   </joint>

Commit message: Fix bno055 driver crash lifecycle, update launch file string parsing, and add static 22-deg tilted LiDAR URDF layout, URDF linked to zero.launch.py

File: src/rover_description/urdf/rover.urdf.xacro (robot description, xacro)
@@ -71,4 +71,6 @@
     <parent link="base_link"/>
     <child link="rslidar"/>
+    <!-- <origin xyz="0.0 0.043684 .19576183" rpy="0 ${-22 * pi / 180} 0"/> -->
+    <!-- <origin xyz="0.0 0.043684 .19576183" rpy="${pi} 0 0"/> -->
     <origin xyz="0.0 0.043684 .19576183" rpy="0 ${22 * pi / 180} 0"/>
   </joint>

File: src/roverrobotics_ros2/roverrobotics_description/urdf/rover_4wd.urdf (robot description, URDF)
Before this commit: robot rover_4wd, 6 links, 5 joints
Links:
- removed link chassis_link
- removed link fl_wheel_link
- removed link fr_wheel_link
- removed link rl_wheel_link
- removed link rr_wheel_link
- added link base_footprint
- added link bno055; visual box size=0.03 0.02 0.01
- added link camera_link; visual box size=0.02 0.06 0.02
- added link camera_link_optical
- added link front_left_wheel; visual cylinder length=0.05 radius=0.1
- added link front_right_wheel; visual cylinder length=0.05 radius=0.1
- added link rear_left_wheel; visual cylinder length=0.05 radius=0.1
- added link rear_right_wheel; visual cylinder length=0.05 radius=0.1
- added link rslidar; visual cylinder length=0.038040 radius=0.061331
- link base_link: geometry visual box size=0.5 0.4 0.25
Joints:
- removed joint base_to_chassis
- removed joint fl_wheel_to_chassis
- removed joint fr_wheel_to_chassis
- removed joint rl_wheel_to_chassis
- removed joint rr_wheel_to_chassis
- added joint base_joint: type fixed, parent base_footprint, child base_link, origin xyz=0 0 0.15000000000000002 rpy=0 0 0
- added joint camera_joint: type fixed, parent base_link, child camera_link, origin xyz=.196296 .060 .135925 rpy=0 0 0
- added joint camera_optical_joint: type fixed, parent camera_link, child camera_link_optical, origin xyz=0 0 0 rpy=-1.5707963267948966 0 -1.5707963267948966
- added joint front_left_wheel_joint: type continuous, parent base_link, child front_left_wheel, origin xyz=0.18 0.225 -0.05 rpy=0 0 0, axis 0 1 0
- added joint front_right_wheel_joint: type continuous, parent base_link, child front_right_wheel, origin xyz=0.18 -0.225 -0.05 rpy=0 0 0, axis 0 1 0
- added joint imu_joint: type fixed, parent base_link, child bno055, origin xyz=-0.03928461 -0.050864 0.14345 rpy=0 0 0
- added joint lidar_joint: type fixed, parent base_link, child rslidar, origin xyz=0.0 0.043684 .19576183 rpy=0 0.3839724354387525 0
- added joint rear_left_wheel_joint: type continuous, parent base_link, child rear_left_wheel, origin xyz=-0.18 0.225 -0.05 rpy=0 0 0, axis 0 1 0
- added joint rear_right_wheel_joint: type continuous, parent base_link, child rear_right_wheel, origin xyz=-0.18 -0.225 -0.05 rpy=0 0 0, axis 0 1 0

Commit message: Corrected base link height WRT ground link

File: src/rover_description/urdf/rover.urdf.xacro (robot description, xacro)
@@ -23,5 +23,6 @@
     <parent link="base_footprint"/>
     <child link="base_link"/>
-    <origin xyz="0 0 ${wheel_radius - wheel_offset_z}" rpy="0 0 0"/>
+    <!-- <origin xyz="0 0 ${wheel_radius - wheel_offset_z}" rpy="0 0 0"/> -->
+    <origin xyz="0 0 0.072" rpy="0 0 0"/>
   </joint>
   <xacro:macro name="wheel" params="prefix x_reflect y_reflect">

File: src/roverrobotics_ros2/roverrobotics_description/urdf/rover_4wd.urdf (robot description, URDF)
Before this commit: robot rover, 10 links, 9 joints
Joints:
- joint base_joint: origin xyz=0 0 0.15000000000000002 rpy=0 0 0 -> xyz=0 0 0.072 rpy=0 0 0
