Commit message: changed urdf to reflect new forward facing payload

File: src/roverrobotics_description/urdf/rover.urdf.xacro (robot description, xacro)
@@ -58,6 +58,6 @@
     <child link="bno055"/>
     <!-- This configuration is based on my estimate for where the center of the chip is
-    the IMU is mounted in a right-handed X right Y forward configuration. -->
-    <origin xyz="-0.03928461 -0.050864 0.14345" rpy="0 0 ${pi/2}"/>
+    the IMU is mounted in a right-handed X forward Y left configuration. -->
+    <origin xyz="0.092487 -0.036660 0.143350" rpy="0 0 0"/>
   </joint>
   <link name="rslidar">
@@ -74,5 +74,5 @@
     <!-- <origin xyz="0.0 0.043684 .19576183" rpy="0 ${-22 * pi / 180} 0"/> -->
     <!-- <origin xyz="0.0 0.043684 .19576183" rpy="${pi} 0 0"/> -->
-    <origin xyz="0.0 0.043684 .19576183" rpy="0 ${22 * pi / 180} 0"/>
+    <origin xyz="0.077296 0.0355 .203479" rpy="0 ${22 * pi / 180} 0"/>
   </joint>
   <link name="camera_link">
@@ -87,5 +87,5 @@
     <parent link="base_link"/>
     <child link="camera_link"/>
-    <origin xyz=".196296 .060 .135925" rpy="0 0 0"/>
+    <origin xyz=".180006 .060 .135925" rpy="0 0 0"/>
   </joint>
   <link name="camera_link_optical"/>

File: src/roverrobotics_description/urdf/rover_4wd.urdf (robot description, URDF)
Before this commit: robot rover, 10 links, 9 joints
Joints:
- joint camera_joint: origin xyz=.196296 .060 .135925 rpy=0 0 0 -> xyz=.180006 .060 .135925 rpy=0 0 0
- joint imu_joint: origin xyz=-0.03928461 -0.050864 0.14345 rpy=0 0 0 -> xyz=0.092487 -0.036660 0.143350 rpy=0 0 0
- joint lidar_joint: origin xyz=0.0 0.043684 .19576183 rpy=0 0.3839724354387525 0 -> xyz=0.077296 0.0355 .203479 rpy=0 0.3839724354387525 0
