Commit message: Updated URDF for new 1650 compliant payload

File: src/roverrobotics_description/urdf/rover_4wd.urdf (robot description, URDF)
Before this commit: robot rover, 9 links, 8 joints
Joints:
- joint imu_joint: origin xyz=0.092487 -0.036660 0.143350 rpy=0 0 0 -> xyz=0.10286227 0.48285 0.141350 rpy=0 0 1.5707963
- joint lidar_joint: origin xyz=0.077296 0.0355 .203479 rpy=0 0.3839724354387525 0 -> xyz=0.158968 0.0 .170481 rpy=0 0.3839724354387525 0
